File: Env-KB60.kicad_pcb (KiCad board)
At the start: 2 copper layers, 286 x 100 mm, 129 parts, among them U1 Pico

Commit message: Added 6*M2 Mount holes
There is one mount hole in each corner and also a couple along the center line of the board, one below the space bar and the other between the top two rows.
Parts:
- added H1: MountingHole, MountingHole:MountingHole_2.2mm_M2, F.Cu at (71.0, 77.0)
- added H2: MountingHole, MountingHole:MountingHole_2.2mm_M2, F.Cu at (71.0, 171.0)
- added H3: MountingHole, MountingHole:MountingHole_2.2mm_M2, F.Cu at (351.0, 171.0)
- added H4: MountingHole, MountingHole:MountingHole_2.2mm_M2, F.Cu at (351.0, 77.0)
- added H5: MountingHole, MountingHole:MountingHole_2.2mm_M2, F.Cu at (211.0, 99.5)
- added H6: MountingHole, MountingHole:MountingHole_2.2mm_M2, F.Cu at (211.0, 171.0)
Routing:
- net row0: track 428.3 -> 424.7 mm
- net row3: track 487.9 -> 486.2 mm
- net gnd: vias 8 -> 9
Other:
- board text added: "https://github.com/Envious-Data/Env-KB60"
