File: Env-KB60.kicad_pcb (KiCad board)
At the start: 2 copper layers, 286 x 100 mm, 135 parts, among them U1 Pico

Commit message: Re-Doing this PCB
Parts:
- removed the D_11 at (276.0, 83.0)
- removed the D_29 at (100.4, 122.2)
- removed the D_43 at (89.5, 152.6)
- removed D_63: D, Diode_THT:D_DO-35_SOD27_P7.62mm_Horizontal
- removed H1, H2, H3, H4, H5, H6: MountingHole, MountingHole:MountingHole_2.2mm_M2
- removed the K_1 at (77.6, 86.9)
- removed the K_29 at (84.8, 125.0)
- removed the K_42 at (332.4, 125.0)
- removed the K_44 at (89.5, 144.1)
- removed the K_57 at (327.7, 144.1)
- removed U1: Pico, MCU_RaspberryPi_and_Boards:RPi_Pico_SMD_TH
- added D_10: D, Diode_SMD:D_SOD-123, B.Cu at (287.6, 50.0)
- added D_40: D, Diode_SMD:D_SOD-123, B.Cu at (339.9, 88.1)
- added D_61: D, Diode_SMD:D_SOD-123, B.Cu at (361.5, 126.2)
- added K_0: KEYSW, MX_Only:MXOnly-1U-NoLED, F.Cu at (88.5, 46.5)
- added K_53: KEYSW, MX_Only:MXOnly-2.75U-NoLED, F.Cu at (338.6, 103.7)
- D_0: renamed from D_1; footprint Diode_THT:D_DO-35_SOD27_P7.62mm_Horizontal -> Diode_SMD:D_SOD-123; moved to B.Cu
- D_1: renamed from D_2; footprint Diode_THT:D_DO-35_SOD27_P7.62mm_Horizontal -> Diode_SMD:D_SOD-123; moved to B.Cu
- D_11: renamed from D_12; footprint Diode_THT:D_DO-35_SOD27_P7.62mm_Horizontal -> Diode_SMD:D_SOD-123; moved to B.Cu
- D_12: renamed from D_13; footprint Diode_THT:D_DO-35_SOD27_P7.62mm_Horizontal -> Diode_SMD:D_SOD-123; moved to B.Cu
- D_13: renamed from D_14; footprint Diode_THT:D_DO-35_SOD27_P7.62mm_Horizontal -> Diode_SMD:D_SOD-123; moved to B.Cu
- D_14: renamed from D_16; footprint Diode_THT:D_DO-35_SOD27_P7.62mm_Horizontal -> Diode_SMD:D_SOD-123; moved to B.Cu
- D_15: renamed from D_17; footprint Diode_THT:D_DO-35_SOD27_P7.62mm_Horizontal -> Diode_SMD:D_SOD-123; moved to B.Cu
- D_16: renamed from D_18; footprint Diode_THT:D_DO-35_SOD27_P7.62mm_Horizontal -> Diode_SMD:D_SOD-123; moved to B.Cu
- D_17: renamed from D_19; footprint Diode_THT:D_DO-35_SOD27_P7.62mm_Horizontal -> Diode_SMD:D_SOD-123; moved to B.Cu
- D_18: renamed from D_20; footprint Diode_THT:D_DO-35_SOD27_P7.62mm_Horizontal -> Diode_SMD:D_SOD-123; moved to B.Cu
- D_19: renamed from D_21; footprint Diode_THT:D_DO-35_SOD27_P7.62mm_Horizontal -> Diode_SMD:D_SOD-123; moved to B.Cu
- D_2: renamed from D_3; footprint Diode_THT:D_DO-35_SOD27_P7.62mm_Horizontal -> Diode_SMD:D_SOD-123; moved to B.Cu
- D_20: renamed from D_22; footprint Diode_THT:D_DO-35_SOD27_P7.62mm_Horizontal -> Diode_SMD:D_SOD-123; moved to B.Cu
- D_21: renamed from D_23; footprint Diode_THT:D_DO-35_SOD27_P7.62mm_Horizontal -> Diode_SMD:D_SOD-123; moved to B.Cu
- D_22: renamed from D_24; footprint Diode_THT:D_DO-35_SOD27_P7.62mm_Horizontal -> Diode_SMD:D_SOD-123; moved to B.Cu
- D_23: renamed from D_25; footprint Diode_THT:D_DO-35_SOD27_P7.62mm_Horizontal -> Diode_SMD:D_SOD-123; moved to B.Cu
- D_24: renamed from D_26; footprint Diode_THT:D_DO-35_SOD27_P7.62mm_Horizontal -> Diode_SMD:D_SOD-123; moved to B.Cu
- D_25: renamed from D_27; footprint Diode_THT:D_DO-35_SOD27_P7.62mm_Horizontal -> Diode_SMD:D_SOD-123; moved to B.Cu
- D_26: renamed from D_15; footprint Diode_THT:D_DO-35_SOD27_P7.62mm_Horizontal -> Diode_SMD:D_SOD-123; moved to B.Cu
- D_27: renamed from D_42; footprint Diode_THT:D_DO-35_SOD27_P7.62mm_Horizontal -> Diode_SMD:D_SOD-123; moved to B.Cu
- D_28, D_41: footprint Diode_THT:D_DO-35_SOD27_P7.62mm_Horizontal -> Diode_SMD:D_SOD-123; moved to B.Cu
- D_29: renamed from D_30; footprint Diode_THT:D_DO-35_SOD27_P7.62mm_Horizontal -> Diode_SMD:D_SOD-123; moved to B.Cu
- D_3: renamed from D_4; footprint Diode_THT:D_DO-35_SOD27_P7.62mm_Horizontal -> Diode_SMD:D_SOD-123; moved to B.Cu
- D_30: renamed from D_31; footprint Diode_THT:D_DO-35_SOD27_P7.62mm_Horizontal -> Diode_SMD:D_SOD-123; moved to B.Cu
- D_31: renamed from D_32; footprint Diode_THT:D_DO-35_SOD27_P7.62mm_Horizontal -> Diode_SMD:D_SOD-123; moved to B.Cu
- D_32: renamed from D_33; footprint Diode_THT:D_DO-35_SOD27_P7.62mm_Horizontal -> Diode_SMD:D_SOD-123; moved to B.Cu
- D_33: renamed from D_34; footprint Diode_THT:D_DO-35_SOD27_P7.62mm_Horizontal -> Diode_SMD:D_SOD-123; moved to B.Cu
- D_34: renamed from D_35; footprint Diode_THT:D_DO-35_SOD27_P7.62mm_Horizontal -> Diode_SMD:D_SOD-123; moved to B.Cu
- D_35: renamed from D_36; footprint Diode_THT:D_DO-35_SOD27_P7.62mm_Horizontal -> Diode_SMD:D_SOD-123; moved to B.Cu
- D_36: renamed from D_37; footprint Diode_THT:D_DO-35_SOD27_P7.62mm_Horizontal -> Diode_SMD:D_SOD-123; moved to B.Cu
- D_37: renamed from D_38; footprint Diode_THT:D_DO-35_SOD27_P7.62mm_Horizontal -> Diode_SMD:D_SOD-123; moved to B.Cu
- D_38: renamed from D_39; footprint Diode_THT:D_DO-35_SOD27_P7.62mm_Horizontal -> Diode_SMD:D_SOD-123; moved to B.Cu
- D_39: renamed from D_40; footprint Diode_THT:D_DO-35_SOD27_P7.62mm_Horizontal -> Diode_SMD:D_SOD-123; moved to B.Cu
- D_4: renamed from D_5; footprint Diode_THT:D_DO-35_SOD27_P7.62mm_Horizontal -> Diode_SMD:D_SOD-123; moved to B.Cu
- D_42: renamed from D_44; footprint Diode_THT:D_DO-35_SOD27_P7.62mm_Horizontal -> Diode_SMD:D_SOD-123; moved to B.Cu
- D_43: renamed from D_45; footprint Diode_THT:D_DO-35_SOD27_P7.62mm_Horizontal -> Diode_SMD:D_SOD-123; moved to B.Cu
- D_44: renamed from D_46; footprint Diode_THT:D_DO-35_SOD27_P7.62mm_Horizontal -> Diode_SMD:D_SOD-123; moved to B.Cu
- D_45: renamed from D_47; footprint Diode_THT:D_DO-35_SOD27_P7.62mm_Horizontal -> Diode_SMD:D_SOD-123; moved to B.Cu
- D_46: renamed from D_48; footprint Diode_THT:D_DO-35_SOD27_P7.62mm_Horizontal -> Diode_SMD:D_SOD-123; moved to B.Cu
- D_47: renamed from D_49; footprint Diode_THT:D_DO-35_SOD27_P7.62mm_Horizontal -> Diode_SMD:D_SOD-123; moved to B.Cu
- D_48: renamed from D_50; footprint Diode_THT:D_DO-35_SOD27_P7.62mm_Horizontal -> Diode_SMD:D_SOD-123; moved to B.Cu
- D_49: renamed from D_51; footprint Diode_THT:D_DO-35_SOD27_P7.62mm_Horizontal -> Diode_SMD:D_SOD-123; moved to B.Cu
- D_5: renamed from D_6; footprint Diode_THT:D_DO-35_SOD27_P7.62mm_Horizontal -> Diode_SMD:D_SOD-123; moved to B.Cu
- D_50: renamed from D_52; footprint Diode_THT:D_DO-35_SOD27_P7.62mm_Horizontal -> Diode_SMD:D_SOD-123; moved to B.Cu
- D_51: renamed from D_53; footprint Diode_THT:D_DO-35_SOD27_P7.62mm_Horizontal -> Diode_SMD:D_SOD-123; moved to B.Cu
- D_52: renamed from D_54; footprint Diode_THT:D_DO-35_SOD27_P7.62mm_Horizontal -> Diode_SMD:D_SOD-123; moved to B.Cu
- D_53: renamed from D_55; footprint Diode_THT:D_DO-35_SOD27_P7.62mm_Horizontal -> Diode_SMD:D_SOD-123; moved to B.Cu
- D_54: renamed from D_56; footprint Diode_THT:D_DO-35_SOD27_P7.62mm_Horizontal -> Diode_SMD:D_SOD-123; moved to B.Cu
- D_55: renamed from D_57; footprint Diode_THT:D_DO-35_SOD27_P7.62mm_Horizontal -> Diode_SMD:D_SOD-123; moved to B.Cu
- D_56: renamed from D_58; footprint Diode_THT:D_DO-35_SOD27_P7.62mm_Horizontal -> Diode_SMD:D_SOD-123; moved to B.Cu
- D_57: renamed from D_59; footprint Diode_THT:D_DO-35_SOD27_P7.62mm_Horizontal -> Diode_SMD:D_SOD-123; moved to B.Cu
- D_58: renamed from D_60; footprint Diode_THT:D_DO-35_SOD27_P7.62mm_Horizontal -> Diode_SMD:D_SOD-123; moved to B.Cu
- D_59: renamed from D_61; footprint Diode_THT:D_DO-35_SOD27_P7.62mm_Horizontal -> Diode_SMD:D_SOD-123; moved to B.Cu
- D_6: renamed from D_7; footprint Diode_THT:D_DO-35_SOD27_P7.62mm_Horizontal -> Diode_SMD:D_SOD-123; moved to B.Cu
- D_60: renamed from D_62; footprint Diode_THT:D_DO-35_SOD27_P7.62mm_Horizontal -> Diode_SMD:D_SOD-123; moved to B.Cu
- D_7: renamed from D_8; footprint Diode_THT:D_DO-35_SOD27_P7.62mm_Horizontal -> Diode_SMD:D_SOD-123; moved to B.Cu
- D_8: renamed from D_9; footprint Diode_THT:D_DO-35_SOD27_P7.62mm_Horizontal -> Diode_SMD:D_SOD-123; moved to B.Cu
- D_9: renamed from D_10; footprint Diode_THT:D_DO-35_SOD27_P7.62mm_Horizontal -> Diode_SMD:D_SOD-123; moved to B.Cu
- K_28: footprint MX_Only:MXOnly-1.5U-NoLED -> MX_Only:MXOnly-1.75U-NoLED
- K_57: renamed from K_61; footprint MX_Only:MXOnly-6.25U-NoLED -> MX_Only:MXOnly-6.25U-ReversedStabilizers-NoLED
- moved D_26 244.9 mm to (335.2, 69.1), turned to 90 degrees
- moved K_28 244.8 mm to (95.7, 84.6)
- moved D_28 215.4 mm to (111.3, 88.1), turned to 90 degrees
- moved D_41 211.5 mm to (101.8, 107.2), turned to 90 degrees
- moved D_9 46.4 mm to (268.5, 50.0), turned to 90 degrees
- moved D_27 44.9 mm to (361.2, 75.8), turned to 90 degrees
- moved K_27 41.9 mm to (352.8, 75.1)
- moved K_51 41.8 mm to (283.8, 103.7)
- moved K_1 41.8 mm to (107.6, 46.5)
- moved K_2 41.8 mm to (126.6, 46.5)
- moved K_3 41.8 mm to (145.7, 46.5)
- moved K_4 41.8 mm to (164.7, 46.5)
- moved K_41 41.8 mm to (90.9, 103.7)
- moved K_42 41.8 mm to (112.3, 103.7)
- moved K_43 41.8 mm to (131.4, 103.7)
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- renumbered K_2 to K_1, K_11 to K_10, K_12 to K_11, K_13 to K_12, K_14 to K_13, K_15 to K_14, K_16 to K_15, K_17 to K_16, K_18 to K_17, K_19 to K_18, K_20 to K_19, K_3 to K_2, K_21 to K_20, K_22 to K_21, K_23 to K_22, K_24 to K_23, K_25 to K_24, K_26 to K_25, K_27 to K_26, K_43 to K_27, K_30 to K_29, K_4 to K_3, K_31 to K_30, K_32 to K_31, K_33 to K_32, K_34 to K_33, K_35 to K_34, K_36 to K_35, K_37 to K_36, K_38 to K_37, K_39 to K_38, K_40 to K_39, K_5 to K_4, K_41 to K_40, K_45 to K_41, K_46 to K_42, K_47 to K_43, K_48 to K_44, K_49 to K_45, K_50 to K_46, K_51 to K_47, K_52 to K_48, K_53 to K_49, K_6 to K_5, K_54 to K_50, K_55 to K_51, K_56 to K_52, K_58 to K_54, K_59 to K_55, K_60 to K_56, K_62 to K_58, K_63 to K_59, K_7 to K_6, K_64 to K_60, K_65 to K_61, K_8 to K_7, K_9 to K_8, K_10 to K_9
Connections:
- D_14 pad 2: Net-(D_16-Pad2) -> Net-(D_14-Pad2)
- D_15 pad 2: Net-(D_17-Pad2) -> Net-(D_15-Pad2)
- D_16 pad 2: Net-(D_18-Pad2) -> Net-(D_16-Pad2)
- D_17 pad 2: Net-(D_19-Pad2) -> Net-(D_17-Pad2)
- D_18 pad 2: Net-(D_20-Pad2) -> Net-(D_18-Pad2)
- D_19 pad 2: Net-(D_21-Pad2) -> Net-(D_19-Pad2)
- D_20 pad 2: Net-(D_22-Pad2) -> Net-(D_20-Pad2)
- D_21 pad 2: Net-(D_23-Pad2) -> Net-(D_21-Pad2)
- D_22 pad 2: Net-(D_24-Pad2) -> Net-(D_22-Pad2)
- D_23 pad 2: Net-(D_25-Pad2) -> Net-(D_23-Pad2)
- D_24 pad 2: Net-(D_26-Pad2) -> Net-(D_24-Pad2)
- D_25 pad 2: Net-(D_27-Pad2) (its old number) -> Net-(D_25-Pad2)
- D_26 pad 2: Net-(D_15-Pad2) -> Net-(D_26-Pad2)
- D_28 pad 1: row1 -> row2
- D_41 pad 1: row2 -> row3
- K_14 pad 2: Net-(D_15-Pad2) -> Net-(D_14-Pad2)
- K_15 pad 2: Net-(D_16-Pad2) -> Net-(D_15-Pad2)
- K_16 pad 2: Net-(D_17-Pad2) -> Net-(D_16-Pad2)
- K_17 pad 2: Net-(D_18-Pad2) -> Net-(D_17-Pad2)
- K_18 pad 2: Net-(D_19-Pad2) -> Net-(D_18-Pad2)
- K_19 pad 2: Net-(D_20-Pad2) -> Net-(D_19-Pad2)
- K_20 pad 2: Net-(D_21-Pad2) -> Net-(D_20-Pad2)
- K_21 pad 2: Net-(D_22-Pad2) -> Net-(D_21-Pad2)
- K_22 pad 2: Net-(D_23-Pad2) -> Net-(D_22-Pad2)
- K_23 pad 2: Net-(D_24-Pad2) -> Net-(D_23-Pad2)
- K_24 pad 2: Net-(D_25-Pad2) -> Net-(D_24-Pad2)
- K_25 pad 2: Net-(D_26-Pad2) -> Net-(D_25-Pad2)
- K_26 pad 2: Net-(D_27-Pad2) (its old number) -> Net-(D_26-Pad2)
- K_28 pad 1: col14 -> col0
- K_40 pad 2: Net-(D_41-Pad2) -> Net-(D_40-Pad2)
- K_41 pad 2: Net-(D_43-Pad2) (its old number) -> Net-(D_41-Pad2)
Routing:
- net row3: track 486.2 -> 0.00 mm
- net col4: track 450.7 -> 0.00 mm
- net row0: track 424.7 -> 0.00 mm
- net row2: track 418.8 -> 0.00 mm
- net row4: track 405.4 -> 0.00 mm
- net row1: track 340.4 -> 0.00 mm
- net col0: track 282.8 -> 0.00 mm
- net col1: track 253.9 -> 0.00 mm
- net col3: track 236.1 -> 0.00 mm
- net col2: track 226.7 -> 0.00 mm
- net col6: track 188.3 -> 0.00 mm
- net col5: track 177.4 -> 0.00 mm
- net col7: track 163.9 -> 0.00 mm
- net col10: track 148.1 -> 0.00 mm
- net col8: track 138.0 -> 0.00 mm
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- removed copper zone on B.Cu, net gnd
- removed copper zone on F.Cu, net gnd
Other:
- board size 286 x 100 mm -> 285 x 94.5 mm
- board text removed: "https://github.com/Envious-Data/Env-KB60"

Commit message: Added Main trace array
Routing:
- net row4: track 0.00 -> 261.0 mm
- net row0: track 0.00 -> 258.2 mm
- net row2: track 0.00 -> 255.0 mm
- net row3: track 0.00 -> 247.5 mm
- net row1: track 0.00 -> 228.6 mm
- net col3: track 0.00 -> 91.8 mm
- net col10: track 0.00 -> 88.3 mm
- net col11: track 0.00 -> 87.7 mm
- net col6: track 0.00 -> 87.5 mm
- net col14: track 0.00 -> 84.7 mm
- net col0: track 0.00 -> 82.0 mm
- net col1: track 0.00 -> 79.2 mm
- net col2: track 0.00 -> 67.6 mm
- net col4: track 0.00 -> 67.5 mm
- net col9: track 0.00 -> 67.5 mm
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
Commit message: Added GH60 compatible mount holes.
Parts:
- added H1: MountingHole, MountingHole:MountingHole_2.5mm, F.Cu at (207.6, 84.5)
- added H2: MountingHole, MountingHole:MountingHole_2.5mm, F.Cu at (339.6, 65.2)
- added H3: MountingHole, MountingHole:MountingHole_2.5mm, F.Cu at (270.0, 122.7)
- added H4: MountingHole, MountingHole:MountingHole_2.5mm, F.Cu at (363.8, 94.1)
- added H5: MountingHole, MountingHole:MountingHole_2.5mm, F.Cu at (80.0, 94.1)
- added H6: MountingHole, MountingHole:MountingHole_2.5mm, F.Cu at (104.7, 65.4)
- K_27: footprint MX_Only:MXOnly-ISO-ROTATED-ReversedStabilizers-NoLED -> MX_Only:MXOnly-ISO-ROTATED
- moved D_14 5.98 mm to (100.6, 69.1)
- moved D_33 5.39 mm to (201.2, 88.1)
- moved D_26 1.18 mm to (334.0, 69.1)
Routing:
- net Net-(D_14-Pad2): track 13.6 -> 8.68 mm
- net row1: track 228.6 -> 233.4 mm
- net Net-(D_33-Pad2): track 9.41 -> 6.90 mm
- net row4: track 261.0 -> 260.3 mm

Commit message: added MCU and some more traces and adjustments
Parts:
- added U1: Pico, MCU_RaspberryPi_and_Boards:RPi_Pico_SMD_TH, B.Cu at (210.0, 120.0)
- D_57: moved to F.Cu
- moved D_57 6.29 mm to (219.0, 120.0)
- moved D_46 1.83 mm to (197.1, 105.3)
- moved D_47 1.83 mm to (216.1, 105.3)
- moved D_48 1.83 mm to (235.2, 105.3)
Routing:
- net row4: track 260.3 -> 271.7 mm, vias 0 -> 2
- net Net-(D_57-Pad2): track 10.1 -> 7.29 mm
- net row3: track 247.5 -> 249.0 mm
- net Net-(D_46-Pad2): track 9.41 -> 8.06 mm
- net Net-(D_48-Pad2): track 9.41 -> 8.12 mm
- net Net-(D_47-Pad2): track 9.41 -> 8.12 mm
- added copper zone on B.Cu, net GND
- added copper zone on F.Cu, net GND
